File: AndromedaV3/AndromedaV3.sch (KiCad schematic (older format))
At the start: 0 parts

Commit message: Add files via upload
Other:
- note added: "1 4"
- note added: "3"
- note added: "6 March 2019"
- note added: "Andromeda V3 by Prithvi Shankara"
Changed lines of the file:
@@
 $Descr A4 11693 8268
 encoding utf-8
-Sheet 1 5
+Sheet 1 4
 Title ""
 Date ""
@@
 $EndSheet
 $Sheet
-S 7500 1800 2300 1500
-U 59D0812B
-F0 "Sensors" 60
-F1 "Peripherals.sch" 60
-$EndSheet
-$Sheet
 S 1875 3875 2250 1525
 U 5A1CBF33
@@
 F1 "Headerssch.sch" 39
 $EndSheet
+Text Notes 7275 7250 0    50   ~ 0
+1 4
+Text Notes 10575 7625 0    50   ~ 0
+3
+Text Notes 7350 7500 0    50   ~ 0
+Andromeda V3 by Prithvi Shankara
+Text Notes 8125 7650 0    50   ~ 0
+6 March 2019
 $EndSCHEMATC
