File: Sensor_Board/Sensor_Board.sch (KiCad schematic (older format))
At the start: 39 parts, among them J1 Micro_SD_Card, J2 Conn_01x08, J3 Conn_01x06, J4 Conn_01x06, J5 Conn_01x06, U1 LSM9DS1, U2 MS5607, U3 ADXL345

Commit message: Add files via upload
Other:
- note added: "1"
- note added: "1 1"
- note added: "6 March 2019"
- note added: "Sensor (Daughter) Board by Prithvi Shankara"
Changed lines of the file:
@@
 	7100 4950 7050 4950
 Connection ~ 7050 4950
+Text Notes 7275 7250 0    50   ~ 0
+1 1
+Text Notes 7350 7500 0    50   ~ 0
+Sensor (Daughter) Board by Prithvi Shankara
+Text Notes 10575 7650 0    50   ~ 0
+1
+Text Notes 8125 7625 0    50   ~ 0
+6 March 2019
 $EndSCHEMATC
